File: kicad/LVGL/TeensyELS.kicad_sch (KiCad schematic)
At the start: 52 parts, among them J1 RJ45_Shielded, J2 Conn_01x04_Pin, J3 Conn_01x14_Socket, J4 Screw_Terminal_01x02, J5 Conn_02x03_Odd_Even, Q1 BSS138, Q2 BSS138, Q3 BSS138, Q4 BSS138, Q5 BSS138, Q6 BSS138, Q7 BSS138, Q8 BSS138, Q9 BSS138, SW1 SW_Omron_B3FS, SW10 SW_Omron_B3FS, SW2 SW_Omron_B3FS, SW3 SW_Omron_B3FS, SW4 SW_Omron_B3FS, SW5 SW_Omron_B3FS, SW6 SW_Omron_B3FS, SW7 SW_Omron_B3FS, SW8 SW_Omron_B3FS, SW9 SW_Omron_B3FS, U1 AMS1117-3.3, U2 ESP32-WROOM-32E

Commit message: Board: fix the R17 pull-up value and publish the production files
Two defects found while tracing the encoder input path through the PCB
netlist for documentation.

R17 was 1K where its counterpart R18 is 10K. They are the pull-ups on the
two channels of one quadrature pair, so there is no reason for them to
differ - it is a slip that got fabricated rather than a design choice. It
works either way, but the 1K draws ten times the current through the
encoder's output transistor. Corrected in the schematic, the board and the
JLCPCB BOM (R17 merges into the existing 10K line, qty 13 -> 14).

No fabrication outputs need regenerating: the value text lives on F.Fab,
which is not among the exported gerber layers, and the silkscreen carries
references only.

kicad/LVGL/jlcpcb/production_files/ was gitignored, so the three files the
README instructs people to order the board from - the only outputs carrying
LCSC part numbers - were never in the repository. Five links in the build
instructions pointed at nothing, while the one BOM that was committed is the
stale kicad/LVGL/production/bom.csv that the README explicitly warns against
using. Un-ignored and committed; the toolkit's project.db and loose gerber
directory stay ignored.

Co-Authored-By: Claude Opus 5 <noreply@anthropic.com>
Claude-Session: https://claude.ai/code/session_01DbAgwqyg5XmoBmuSVBKB19
Parts:
- R17: value 1K -> 10K
Changed lines of the file:
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@@
 			)
 		)
-		(property "Value" "1K"
+		(property "Value" "10K"
 			(at 106.68 194.3099 0)
 			(effects
