File: kicad/LVGL/TeensyELS.kicad_pcb (KiCad board)
At the start: 4 copper layers, 96.6 x 91.3 mm, 58 parts, among them J1 RJ45_Shielded, J2 Conn_01x04_Pin, J3 Conn_01x14_Socket, J4 Screw_Terminal_01x02, J5 Conn_02x03_Odd_Even, Q1 BSS138, Q2 BSS138, Q3 BSS138, Q4 BSS138, Q5 BSS138, Q6 BSS138, Q7 BSS138, Q8 BSS138, Q9 BSS138, SW1 SW_Omron_B3FS, SW10 SW_Omron_B3FS, SW2 SW_Omron_B3FS, SW3 SW_Omron_B3FS, SW4 SW_Omron_B3FS, SW5 SW_Omron_B3FS, SW6 SW_Omron_B3FS, SW7 SW_Omron_B3FS, SW8 SW_Omron_B3FS, SW9 SW_Omron_B3FS, U1 AMS1117-3.3, U2 ESP32-WROOM-32E

Commit message: Board: fix the R17 pull-up value and publish the production files
Two defects found while tracing the encoder input path through the PCB
netlist for documentation.

R17 was 1K where its counterpart R18 is 10K. They are the pull-ups on the
two channels of one quadrature pair, so there is no reason for them to
differ - it is a slip that got fabricated rather than a design choice. It
works either way, but the 1K draws ten times the current through the
encoder's output transistor. Corrected in the schematic, the board and the
JLCPCB BOM (R17 merges into the existing 10K line, qty 13 -> 14).

No fabrication outputs need regenerating: the value text lives on F.Fab,
which is not among the exported gerber layers, and the silkscreen carries
references only.

kicad/LVGL/jlcpcb/production_files/ was gitignored, so the three files the
README instructs people to order the board from - the only outputs carrying
LCSC part numbers - were never in the repository. Five links in the build
instructions pointed at nothing, while the one BOM that was committed is the
stale kicad/LVGL/production/bom.csv that the README explicitly warns against
using. Un-ignored and committed; the toolkit's project.db and loose gerber
directory stay ignored.

Co-Authored-By: Claude Opus 5 <noreply@anthropic.com>
Claude-Session: https://claude.ai/code/session_01DbAgwqyg5XmoBmuSVBKB19
Parts:
- R17: value 1K -> 10K
Changed lines of the file:
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@@
 			)
 		)
-		(property "Value" "1K"
+		(property "Value" "10K"
 			(at 0 1.65 0)
 			(layer "F.Fab")

Commit message: Choose the encoder input type with a jumper, not a soldering iron
R13/R14 were 0R links: fit them and the spindle encoder's A/B arrive straight
on IO34/IO35; leave them off, fit R15/R16 instead, and the signal goes through
the BSS138s. Picking between the two meant a soldering iron and knowing which
of four 0805s in a row did what. J7, an 8-way header, makes it two jumpers.

Which position means what is not readable off the board, so the silkscreen now
carries a legend - the header drawn twice with the shunts shown in place:

* Volt, rows 1 and 3, pads (7,8) and (3,4). Through R16/R15 into the gates of
  Q8/Q1. A 5V or 12V push-pull output must NOT reach IO34/IO35, whose absolute
  maximum is 3.6V; the FETs level-shift it. They also invert it, which for a
  quadrature pair with no index costs nothing - inverting BOTH channels
  preserves which one leads.

* NPN, rows 2 and 4, pads (5,6) and (1,2). Straight through. An open-collector
  output sinks against R18/R17, the 10K pull-ups to +3.3V already on those nets.

FIT ONE SET, NEVER BOTH. With both in on a channel the FET's drain IS the
signal driving its gate, so it shorts the encoder's output to ground every time
that output goes high. The legend draws two whole configurations for exactly
that reason. The old 0R/1K pairs carried the same hazard, but you had to reach
for solder to create it. Note also that the gate is driven through 1K with no
clamp, so "Volt" means up to the BSS138's +/-20V VGS: a 24V encoder is past it.

THE KNOB NOW HAS A BUTTON. E1 pin 3 was unconnected; it goes through R22 (1K)
to IO0, which R20 already pulls to +3.3V, so a press reads about 0.3V. Nothing
in the firmware reads it yet. IO0 is a strapping pin, so holding the knob down
through a reset puts the ESP32 into serial-download mode - a black screen, and
not something firmware can defend against, because the level is latched before
any code runs.

SW1 IS GONE. It shorted the driver side of Q2 to +5V by hand, which is the same
pulse the al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
Parts:
- removed R13, R14: 0K, Resistor_SMD:R_0805_2012Metric
- removed SW1: SW_Omron_B3FS, Button_Switch_SMD:SW_SPST_Omron_B3FS-101xP
- added J7: Conn_02x04_Odd_Even, Connector_PinHeader_2.54mm:PinHeader_2x04_P2.54mm_Vertical, F.Cu at (100.9, 77.7)
- added R22: 1K, Resistor_SMD:R_0805_2012Metric, F.Cu at (95.3, 41.2)
- moved Q1 7.27 mm to (87.0, 77.3)
- moved Q8 7.27 mm to (87.0, 71.3)
- moved R15 7.27 mm to (94.0, 75.3)
- moved R16 7.27 mm to (94.0, 71.3)
- moved R17 7.27 mm to (83.1, 77.3)
- moved R18 7.27 mm to (83.1, 71.3)
Connections:
- E1 pad 3: unconnected-(E1-SW-Pad3) -> Net-(E1-SW)
- R15 pad 1: Net-(J2-Pin_3) -> Net-(J7-Pin_4)
- R16 pad 1: Net-(J2-Pin_4) -> Net-(J7-Pin_8)
Routing:
- net /BOOT: track 57.5 -> 104.7 mm
- net Net-(Q2-D): track 64.8 -> 25.3 mm
- net +5V: track 129.2 -> 109.8 mm
- net /EncA: track 81.1 -> 75.3 mm
- net Net-(J7-Pin_8): track 0.00 -> 4.03 mm
- net Net-(J7-Pin_4): track 0.00 -> 3.58 mm
- net /Blue: track 87.0 -> 83.7 mm
- net Net-(E1-SW): track 0.00 -> 2.94 mm
- net Net-(J2-Pin_3): track 7.79 -> 10.3 mm
- net /EncB: track 77.9 -> 75.9 mm
- net /Ena: track 70.4 -> 68.8 mm
- net /Green: track 26.8 -> 28.2 mm
- net Net-(J2-Pin_4): track 7.59 -> 8.99 mm
- net /UIEncB: track 83.8 -> 82.5 mm
- net /UIEncA: track 79.8 -> 78.8 mm
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Other:
- board text added: "+"
- board text added: "J7"
- board text added: "NPN"
- board text added: "TeensyELS v0.7"
- board text added: "Volt"
- board text removed: "TeensyELS v0.6"

Commit message: The knob switch returns to +5V, so invert it into IO0
1cedd6c wired E1 pin 3 through R22 straight to IO0, on the assumption that the
switch's other terminal was the encoder common, which this board ties to
ground. It is not. It returns to pin 5 - the LED common anode, which sits at
+5V. That commit's account of the circuit is wrong in both directions, and this
corrects it.

WHAT THE COMMITTED CIRCUIT WOULD HAVE DONE. Two failures, neither needing the
other to be fatal:

* IT COULD NOT BE READ. R20 already pulls IO0 to +3.3V, so the pin idles HIGH.
  A press pulls it up as well. Both states are the same state.

* PRESSED WAS OUT OF SPEC. Ignoring the clamp, the node would sit at
  (5/1K + 3.3/10K) / (1/1K + 1/10K) = 4.85V. The ESP32's protection diode pins
  it near 3.9V instead and swallows about 1.1mA into the 3.3V rail. Absolute
  maximum on a GPIO is VDD+0.3 = 3.6V.

The boot warning in that message was backwards too: a press would have held IO0
HIGH, the normal boot level, so it could never have reached download mode.

THE FIX IS THE LEVEL SHIFT THIS BOARD USES EVERYWHERE ELSE. R22 now feeds the
gate of Q10, a BSS138, instead of IO0. R23 (10K) holds that gate down so it
does not float while the switch is open. Q10's source is grounded, its drain is
IO0, and R20 goes on being both the pull-up and the boot strap.

  released   gate at 0V, FET off, IO0 at 3.3V - the level a normal boot needs
  pressed    gate at 4.55V, FET on, IO0 at ~0V

Active low. The gate sits at 4.55V rather than 5V because R22 and R23 divide
it, which is still far above the BSS138's threshold and far below its +/-20V
VGS limit; the switch carries 5V/11K = 455uA.

THE STRAPPING HAZARD IS NOW REAL, where the earlier note only imagined it.
Holding the knob through a reset pulls IO0 low and the ESP32 comes up in serial
download mode - a black screen until it is power-cycled without the knob. That
is ordinary BOOT-button behaviour and it is a deliberate trade, because IO0 is
the only pin left: the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
Parts:
- added Q10: BSS138, Package_TO_SOT_SMD:SOT-23, F.Cu at (86.8, 26.7)
- added R23: 10K, Resistor_SMD:R_0805_2012Metric, F.Cu at (92.1, 27.2)
Connections:
- R22 pad 2: /BOOT -> /KnobSw
Routing:
- net /KnobSw: track 0.00 -> 20.7 mm
- net /BOOT: track 104.7 -> 87.4 mm
- net GND: track 43.3 -> 51.8 mm, vias 11 -> 12

Commit message: Make the programming header a right-angle part, reachable from the edge
J5 was a vertical SMD header sitting on the board face, which means a
programmer can only be plugged in with the board out. It is now the horizontal
variant, moved from (32.53, 24.21) at -90 to (31.38, 26.95) at 90, so the pins
present at the top board edge: the fab outline reaches y=19.67 against an edge
at y=19.90, i.e. flush with it.

IT IS NO LONGER AN SMD PART. Connector_PinHeader_1.27mm has no horizontal SMD
variant, so this is PinHeader_2x03_P1.27mm_Horizontal - six plated holes,
0.65mm drill on 1.0mm pads, where there were six 2.4x0.74mm SMD pads. That
takes J5 out of the SMT placement step and makes it a through-hole line item.
The committed CPL and position files are a rev behind already and will need
regenerating regardless, but this is now a reason rather than just tidiness.

Nets survived pad for pad: 1 /EN, 2 +3.3V, 3 /TXD, 4 GND, 5 /RXD, 6 /BOOT.

The schematic's Footprint field is set to match here. It had already been
changed in eeschema but not yet saved, so the file on disk still named the
Vertical_SMD part at the moment this was checked; saving afterwards produced
byte-identical content, so the two routes agreed and nothing was lost.
Connectivity is untouched and ERC is unmoved at 63. One general note worth
keeping from the confusion: KiCad's schematic-parity check does NOT compare
footprint identity - it reported clean while the two files named different
parts - so a real sch/pcb footprint mismatch will not be caught by DRC.

ONE NEW DRC ERROR, DELIBERATELY LEFT FOR A DECISION: starved_thermal on J5
pad 2 (+3.3V) against the In2.Cu plane - one thermal spoke where the zone asks
for two, because 1.27mm pitch leaves nowhere to put the second. The pad IS
connected; unconnected items are still zero. The choices are to set that pad's
zone connection to solid, to drop the zone's minimum spoke count, or to waive
it, and which one is right depends on how the board gets assembled. Not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
Parts:
- J5: footprint Connector_PinHeader_1.27mm:PinHeader_2x03_P1.27mm_Vertical_SMD -> Connector_PinHeader_1.27mm:PinHeader_2x03_P1.27mm_Horizontal
- moved J5 2.97 mm to (31.4, 26.9), turned to 90 degrees
Routing:
- net /RXD: track 53.0 -> 44.5 mm
- net /TXD: track 49.3 -> 44.4 mm
- net /BOOT: track 87.4 -> 84.3 mm
- net +3.3V: track 72.7 -> 70.5 mm, vias 11 -> 10
- net /EN: track 32.8 -> 30.9 mm, vias 2 -> 0
- net GND: track 51.8 -> 50.6 mm, vias 12 -> 11
